File: Simple BMS Module.kicad_sch (KiCad schematic)
At the start: 11 parts, among them J1 INPUT Voltage, J2 BATTERY, Q1 TIP42C, U1 TL431LP

Commit message: Simple BMS module is renewed
Other:
- company: (none) -> by Muxtar_Safarov
- title: (none) -> Simple BMS Module 
Changed lines of the file:
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@@
 (kicad_sch (version 20230121) (generator eeschema)
   (paper "A4")
+  (title_block
+    (title "Simple BMS Module ")
+    (date "24.03.2023")
+    (rev "1.0")
+    (company "by Muxtar_Safarov")
+  )
   (junction (at 165.1 36.83) (diameter 0) (color 0 0 0 0)
   )
